Commit message: 增加模型文件，修改urdf

File: wheeltec_description/urdf/robot.urdf.xacro (robot description, xacro)
@@ -6,21 +6,20 @@
   <!-- ============================================================ -->
   <!-- 底盘尺寸 -->
-  <xacro:property name="base_length" value="0.30"/>    <!-- 底盘长度 (m) -->
-  <xacro:property name="base_width" value="0.26"/>     <!-- 底盘宽度 (m) -->
-  <xacro:property name="base_height" value="0.10"/>    <!-- 底盘高度 (m) -->
-  <!-- 轮子参数 -->
-  <xacro:property name="wheel_radius" value="0.05"/>   <!-- 轮子半径 (m) -->
-  <xacro:property name="wheel_width" value="0.04"/>    <!-- 轮子宽度 (m) -->
-  <xacro:property name="wheel_separation" value="0.30"/>  <!-- 轮距 (m) -->
-  <xacro:property name="wheel_base" value="0.25"/>     <!-- 轴距 (m) -->
+  <xacro:property name="base_length" value="0.50"/>    <!-- 底盘长度 (m) -->
+  <xacro:property name="base_width" value="0.43"/>     <!-- 底盘宽度 (m) -->
+  <xacro:property name="base_height" value="0.15"/>    <!-- 底盘高度 (m) -->
+  <!-- 轮子参数 (根据 robot_params.hpp 更新) -->
+  <xacro:property name="wheel_radius" value="0.075"/>  <!-- 轮子半径 (m) = 直径0.15/2 -->
+  <xacro:property name="wheel_width" value="0.06"/>    <!-- 轮子宽度 (m) -->
+  <xacro:property name="wheel_separation" value="0.50"/>  <!-- 轮距 (m) -->
+  <xacro:property name="wheel_base" value="0.43"/>     <!-- 轴距 (m) -->
   <!-- 激光雷达安装位置（相对于base_link） -->
-  <!-- TODO: 根据实际安装位置修改 -->
-  <xacro:property name="lidar_x" value="0.0"/>         <!-- X方向偏移 (m) -->
-  <xacro:property name="lidar_y" value="0.0"/>         <!-- Y方向偏移 (m) -->
-  <xacro:property name="lidar_z" value="0.20"/>        <!-- Z方向偏移 (m) -->
+  <xacro:property name="lidar_x" value="-0.20"/>       <!-- X方向偏移 (m) 向后20cm -->
+  <xacro:property name="lidar_y" value="-0.05"/>       <!-- Y方向偏移 (m) 向右5cm -->
+  <xacro:property name="lidar_z" value="0.25"/>        <!-- Z方向偏移 (m) -->
   <!-- IMU安装位置（相对于base_link） -->
   <xacro:property name="imu_x" value="0.0"/>
   <xacro:property name="imu_y" value="0.0"/>
-  <xacro:property name="imu_z" value="0.05"/>
+  <xacro:property name="imu_z" value="0.075"/>
   <!-- ============================================================ -->
   <!-- 材质定义 -->
@@ -38,4 +37,7 @@
     <color rgba="0.8 0.2 0.2 1"/>
   </material>
+  <material name="green">
+    <color rgba="0.2 0.8 0.2 1"/>
+  </material>
   <!-- ============================================================ -->
   <!-- base_footprint - 地面投影坐标系 -->
@@ -52,11 +54,15 @@
   <link name="base_link">
     <visual>
-      <origin xyz="0 0 ${base_height/2}" rpy="0 0 0"/>
+      <!-- 使用 STL 模型文件 -->
+      <!-- 注意: scale="0.001" 表示 STL 单位是 mm，转换为 m -->
+      <!-- Z 轴偏移 +0.075m，绕 Z 轴旋转 90 度 (pi/2 = 1.5708 rad) -->
+      <origin xyz="0 0 0.075" rpy="0 0 1.5708"/>
       <geometry>
-        <box size="${base_length} ${base_width} ${base_height}"/>
+        <mesh filename="package://wheeltec_description/meshes/model3.stl" scale="0.001 0.001 0.001"/>
       </geometry>
-      <material name="grey"/>
+      <material name="green"/>
     </visual>
     <collision>
+      <!-- 碰撞使用简化的盒子模型，提高性能 -->
       <origin xyz="0 0 ${base_height/2}" rpy="0 0 0"/>
       <geometry>
@@ -66,6 +72,6 @@
     <inertial>
       <origin xyz="0 0 ${base_height/2}" rpy="0 0 0"/>
-      <mass value="5.0"/>
-      <inertia ixx="0.05" ixy="0" ixz="0" iyy="0.05" iyz="0" izz="0.05"/>
+      <mass value="10.0"/>
+      <inertia ixx="0.1" ixy="0" ixz="0" iyy="0.1" iyz="0" izz="0.1"/>
     </inertial>
   </link>
@@ -75,11 +81,6 @@
   <xacro:macro name="wheel" params="prefix x_reflect y_reflect">
     <link name="${prefix}_wheel_link">
-      <visual>
-        <origin xyz="0 0 0" rpy="${pi/2} 0 0"/>
-        <geometry>
-          <cylinder radius="${wheel_radius}" length="${wheel_width}"/>
-        </geometry>
-        <material name="black"/>
-      </visual>
+      <!-- 不显示轮子视觉模型，因为 STL 模型已经包含轮子 -->
+      <!-- 只保留碰撞和惯性属性用于物理仿真 -->
       <collision>
         <origin xyz="0 0 0" rpy="${pi/2} 0 0"/>

Commit message: slam建图模式已可用，现在改为同时保存栅格地图和序列化地图；导航模式修改为slam_toolbox 自动定位

File: wheeltec_description/urdf/robot.urdf.xacro (robot description, xacro)
@@ -15,7 +15,8 @@
   <xacro:property name="wheel_base" value="0.43"/>     <!-- 轴距 (m) -->
   <!-- 激光雷达安装位置（相对于base_link） -->
+  <!-- 雷达在车辆后方(-X方向)，距地面30cm（base_link在7.5cm，所以相对Z=22.5cm） -->
   <xacro:property name="lidar_x" value="-0.20"/>       <!-- X方向偏移 (m) 向后20cm -->
-  <xacro:property name="lidar_y" value="-0.05"/>       <!-- Y方向偏移 (m) 向右5cm -->
-  <xacro:property name="lidar_z" value="0.25"/>        <!-- Z方向偏移 (m) -->
+  <xacro:property name="lidar_y" value="0.0"/>         <!-- Y方向偏移 (m) -->
+  <xacro:property name="lidar_z" value="0.225"/>       <!-- Z方向偏移 (m) 距地面30cm -->
   <!-- IMU安装位置（相对于base_link） -->
   <xacro:property name="imu_x" value="0.0"/>
@@ -133,5 +134,6 @@
     <parent link="base_link"/>
     <child link="laser_frame"/>
-    <origin xyz="${lidar_x} ${lidar_y} ${lidar_z}" rpy="0 0 0"/>
+    <!-- X轴旋转180度修复上下颠倒，Z轴旋转180度调整扫描方向 -->
+    <origin xyz="${lidar_x} ${lidar_y} ${lidar_z}" rpy="${pi} 0 ${pi}"/>
   </joint>
   <!-- ============================================================ -->

Commit message: fix(driver): 修正底盘速度比例因子并优化 Nav2 DWB 参数
1. 修正驱动层速度转换倍率：
   - 经实测，底盘协议的最小速度单位约为 0.2857 m/s。
   - 将 serial_protocol.hpp 中的缩放因子调整为 3.5 (1.0 / 0.2857)，并增加 std::round 取整。
   - 解决了 ROS 层发送 1.0 m/s 指令时底层速度过小或为 0 的问题。

2. 优化 Nav2 参数配置 (nav2_params.yaml)：
   - 恢复加速度限制为标准值 (2.5 m/s²)，移除调试用的激进参数 (20.0 m/s²)。
   - 恢复最小速度限制为 0.0，允许低速平滑运行。
   - 调整 DWB Local Planner：
     - 禁用 PathAlign 和 GoalAlign (scale设为0.0)，允许麦轮底盘全向移动，无需强制旋转对齐路径。
     - 降低 RotateToGoal 权重，优先保证位移速度。
     - 调整采样数 (samples=15) 以平衡 CPU 负载和路径搜索质量。

File: wheeltec_description/urdf/robot.urdf.xacro (robot description, xacro)
@@ -17,5 +17,5 @@
   <!-- 雷达在车辆后方(-X方向)，距地面30cm（base_link在7.5cm，所以相对Z=22.5cm） -->
   <xacro:property name="lidar_x" value="-0.20"/>       <!-- X方向偏移 (m) 向后20cm -->
-  <xacro:property name="lidar_y" value="0.0"/>         <!-- Y方向偏移 (m) -->
+  <xacro:property name="lidar_y" value="0.0"/>         <!-- Y方向偏移 (m) 实际偏右5cm，但需匹配建图时TF，重建图后改为-0.05 -->
   <xacro:property name="lidar_z" value="0.225"/>       <!-- Z方向偏移 (m) 距地面30cm -->
   <!-- IMU安装位置（相对于base_link） -->
@@ -134,5 +134,5 @@
     <parent link="base_link"/>
     <child link="laser_frame"/>
-    <!-- X轴旋转180度修复上下颠倒，Z轴旋转180度调整扫描方向 -->
+    <!-- X轴旋转180度修正Z轴方向，Z轴旋转180度匹配雷达安装方向 -->
     <origin xyz="${lidar_x} ${lidar_y} ${lidar_z}" rpy="${pi} 0 ${pi}"/>
   </joint>
